Commit message: Added the bot node to world launch and fixed a bug

File: src/my_robot/urdf/my_robot.xacro (robot description, xacro)
@@ -114,5 +114,5 @@
     <child link="right_wheel"/>
     <parent link="chassis"/>
-    <axis xyz="0 -1 0" rpy="0 0 0"/>
+    <axis xyz="0 1 0" rpy="0 0 0"/>
     <limit effort="10000" velocity="1000"/>
     <dynamics damping="1.0" friction="1.0"/>
